Commit message: added hokuyo scanner

File: robots/youbot.urdf.xacro (robot description, xacro)
@@ -3,5 +3,5 @@
        xmlns:controller="http://playerstage.sourceforge.net/gazebo/xmlschema/#controller"
        xmlns:interface="http://playerstage.sourceforge.net/gazebo/xmlschema/#interface"
-       xmlns:xacro="http://playerstage.sourceforge.net/gazebo/xmlschema/#interface"
+       xmlns:xacro="http://ros.org/wiki/xacro"
        name="youbot" >
   <!-- The following xacro:included files set up definitions of parts of the robot body -->

File: robots/youbot_arm_only.urdf.xacro (robot description, xacro)
@@ -3,5 +3,5 @@
        xmlns:controller="http://playerstage.sourceforge.net/gazebo/xmlschema/#controller"
        xmlns:interface="http://playerstage.sourceforge.net/gazebo/xmlschema/#interface"
-       xmlns:xacro="http://playerstage.sourceforge.net/gazebo/xmlschema/#interface"
+       xmlns:xacro="http://ros.org/wiki/xacro"
        name="youbot" >
   <!-- The following included files set up definitions of parts of the robot body -->

File: robots/youbot_base_only.urdf.xacro (robot description, xacro)
@@ -3,5 +3,5 @@
        xmlns:controller="http://playerstage.sourceforge.net/gazebo/xmlschema/#controller"
        xmlns:interface="http://playerstage.sourceforge.net/gazebo/xmlschema/#interface"
-       xmlns:xacro="http://playerstage.sourceforge.net/gazebo/xmlschema/#interface"
+       xmlns:xacro="http://ros.org/wiki/xacro"
        name="youbot" >
   <!-- The following xacro:included files set up definitions of parts of the robot body -->

File: robots/youbot_dual_arm.urdf.xacro (robot description, xacro)
@@ -3,5 +3,5 @@
        xmlns:controller="http://playerstage.sourceforge.net/gazebo/xmlschema/#controller"
        xmlns:interface="http://playerstage.sourceforge.net/gazebo/xmlschema/#interface"
-       xmlns:xacro="http://playerstage.sourceforge.net/gazebo/xmlschema/#interface"
+       xmlns:xacro="http://ros.org/wiki/xacro"
        name="youbot" >
   <!-- The following xacro:included files set up definitions of parts of the robot body -->

File: urdf/common.xacro (robot description, xacro)
@@ -1,9 +1,9 @@
 <?xml version="1.0"?>
-<robot>
-	<property name="M_PI" value="3.1415926535897931" />
+<robot xmlns:xacro="http://ros.org/wiki/xacro">
+	<xacro:property name="M_PI" value="3.1415926535897931" />
 	<!-- Casters -->
-	<property name="cal_caster_fl" value="0.0" />
-	<property name="cal_caster_fr" value="0.0" />
-	<property name="cal_caster_bl" value="0.0" />
-	<property name="cal_caster_br" value="0.0" />
+	<xacro:property name="cal_caster_fl" value="0.0" />
+	<xacro:property name="cal_caster_fr" value="0.0" />
+	<xacro:property name="cal_caster_bl" value="0.0" />
+	<xacro:property name="cal_caster_br" value="0.0" />
 </robot>

File: urdf/misc/cam3d_tower.urdf.xacro (robot description, xacro)
@@ -4,7 +4,7 @@
        xmlns:interface="http://playerstage.sourceforge.net/gazebo/xmlschema/#interface"
        xmlns:xacro="http://ros.org/wiki/xacro">
-  <property name="cam3d_tower_height" value="0.49" />
-  <property name="cam3d_tower_width" value="0.03" />
-  <property name="cam3d_tower_depth" value="0.03" />
+  <xacro:property name="cam3d_tower_height" value="0.49" />
+  <xacro:property name="cam3d_tower_width" value="0.03" />
+  <xacro:property name="cam3d_tower_depth" value="0.03" />
   <xacro:macro name="cam3d_tower" params="name parent *origin">
   	<link name="${name}_link">
@@ -29,5 +29,5 @@
     </link>
     <joint name="${name}_joint" type="fixed">
-      <insert_block name="origin" />
+      <xacro:insert_block name="origin" />
       <parent link="${parent}"/>
       <child link="${name}_link"/>

File: urdf/misc/sensor_angle.urdf.xacro (robot description, xacro)
@@ -4,7 +4,7 @@
        xmlns:interface="http://playerstage.sourceforge.net/gazebo/xmlschema/#interface"
        xmlns:xacro="http://ros.org/wiki/xacro">
-	<property name="sensor_angle_width"  value="0.097" />
-	<property name="sensor_angle_height" value="0.0015" />
-	<property name="sensor_angle_depth"  value="0.0625" />
+	<xacro:property name="sensor_angle_width"  value="0.097" />
+	<xacro:property name="sensor_angle_height" value="0.0015" />
+	<xacro:property name="sensor_angle_depth"  value="0.0625" />
 	<xacro:macro name="sensor_angle" params="name parent *origin">
 		<link name="${name}_part1_link">
@@ -29,5 +29,5 @@
 		</link>
 		<joint name="${name}_part1_joint" type="fixed">
-			<insert_block name="origin" />
+			<xacro:insert_block name="origin" />
 			<parent link="${parent}"/>
 			<child link="${name}_part1_link"/>

File: urdf/sensors/hokuyo_urg04_laser.urdf.xacro (robot description, xacro)
@@ -8,5 +8,5 @@
     <joint name="${name}_hokuyo_urg04_laser_joint" type="fixed">
       <axis xyz="0 1 0" />
-      <insert_block name="origin" />
+      <xacro:insert_block name="origin" />
       <parent link="${parent}_link"/>
       <child link="${name}_link"/>

File: urdf/youbot_arm/arm.transmission.xacro (robot description, xacro)
@@ -8,52 +8,52 @@
 	<xacro:macro name="youbot_arm_transmission" params="name">
 		<transmission name="${name}_trans_1">
-			<type>transmission_interface/SimpleTransmission</type>
+      <type>transmission_interface/SimpleTransmission</type>
 			<actuator name="${name}_motor_1">
-				<hardwareInterface>EffortJointInterface</hardwareInterface>
-				<mechanicalReduction>1</mechanicalReduction>
-			</actuator>
+        <hardwareInterface>EffortJointInterface</hardwareInterface>
+        <mechanicalReduction>1</mechanicalReduction>
+      </actuator>
 			<joint name="${name}_joint_1">
-				<hardwareInterface>EffortJointInterface</hardwareInterface>
-			</joint>
+        <hardwareInterface>EffortJointInterface</hardwareInterface>
+      </joint>
 		</transmission>
 		<transmission name="${name}_trans_2">
-			<type>transmission_interface/SimpleTransmission</type>
+      <type>transmission_interface/SimpleTransmission</type>
 			<actuator name="${name}_motor_2">
-				<hardwareInterface>EffortJointInterface</hardwareInterface>
-				<mechanicalReduction>1</mechanicalReduction>
-			</actuator>
+        <hardwareInterface>EffortJointInterface</hardwareInterface>
+        <mechanicalReduction>1</mechanicalReduction>
+      </actuator>
 			<joint name="${name}_joint_2">
-				<hardwareInterface>EffortJointInterface</hardwareInterface>
-			</joint>
+        <hardwareInterface>EffortJointInterface</hardwareInterface>
+      </joint>
 		</transmission>
 		<transmission name="${name}_trans_3">
-			<type>transmission_interface/SimpleTransmission</type>
+      <type>transmission_interface/SimpleTransmission</type>
 			<actuator name="${name}_motor_3">
-				<hardwareInterface>EffortJointInterface</hardwareInterface>
-				<mechanicalReduction>1</mechanicalReduction>
-			</actuator>
+        <hardwareInterface>EffortJointInterface</hardwareInterface>
+        <mechanicalReduction>1</mechanicalReduction>
+      </actuator>
 			<joint name="${name}_joint_3">
-				<hardwareInterface>EffortJointInterface</hardwareInterface>
-			</joint>
+        <hardwareInterface>EffortJointInterface</hardwareInterface>
+      </joint>
 		</transmission>
 		<transmission name="${name}_trans_4">
-			<type>transmission_interface/SimpleTransmission</type>
+      <type>transmission_interface/SimpleTransmission</type>
 			<actuator name="${name}_motor_4">
-				<hardwareInterface>EffortJointInterface</hardwareInterface>
-				<mechanicalReduction>1</mechanicalReduction>
-			</actuator>
+        <hardwareInterface>EffortJointInterface</hardwareInterface>
+        <mechanicalReduction>1</mechanicalReduction>
+      </actuator>
 			<joint name="${name}_joint_4">
-				<hardwareInterface>EffortJointInterface</hardwareInterface>
-			</joint>
+        <hardwareInterface>EffortJointInterface</hardwareInterface>
+      </joint>
 		</transmission>
 		<transmission name="${name}_trans_5">
-			<type>transmission_interface/SimpleTransmission</type>
+      <type>transmission_interface/SimpleTransmission</type>
 			<actuator name="${name}_motor_5">
-				<hardwareInterface>EffortJointInterface</hardwareInterface>
-				<mechanicalReduction>1</mechanicalReduction>
-			</actuator>
+        <hardwareInterface>EffortJointInterface</hardwareInterface>
+        <mechanicalReduction>1</mechanicalReduction>
+      </actuator>
 			<joint name="${name}_joint_5">
-				<hardwareInterface>EffortJointInterface</hardwareInterface>
-			</joint>
+        <hardwareInterface>EffortJointInterface</hardwareInterface>
+      </joint>
 		</transmission>
 	</xacro:macro>

File: urdf/youbot_arm/arm.urdf.xacro (robot description, xacro)
@@ -10,5 +10,5 @@
 		<!-- joint between base_link and arm_0_link -->
 		<joint name="${name}_joint_0" type="fixed" >
-			<insert_block name="origin" />
+			<xacro:insert_block name="origin" />
 			<parent link="${parent}" />
 			<child link="${name}_link_0" />

File: urdf/youbot_arm/limits.urdf.xacro (robot description, xacro)
@@ -2,30 +2,30 @@
 <robot xmlns:xacro="http://ros.org/wiki/xacro">>
 	<!-- common properties -->
-	<property name="M_PI" value="3.1415926535897931" />
-        <property name="threshold" value="0.01" />
+	<xacro:property name="M_PI" value="3.1415926535897931" />
+        <xacro:property name="threshold" value="0.01" />
 	<!-- arm limits positions (deg) -->
-	<property name="joint_1_limit" value="${M_PI * (169 + 169) / 180}" />
-	<property name="joint_2_limit" value="${M_PI * (90 + 65) / 180}" />
-	<property name="joint_3_limit" value="${M_PI * (146 + 151) / 180}" />
-	<property name="joint_4_limit" value="${M_PI * (102.5 + 102.5) / 180}" />
-	<property name="joint_5_limit" value="${M_PI * (167.5 + 167.5) / 180}" />
-        <property name="joint_1_limit_soft" value="${M_PI * (169 + 169) / 180 - threshold}" />
-	<property name="joint_2_limit_soft" value="${M_PI * (90 + 65) / 180 - threshold}" />
-	<property name="joint_3_limit_soft" value="${M_PI * (146 + 151) / 180 - threshold}" />
-	<property name="joint_4_limit_soft" value="${M_PI * (102.5 + 102.5) / 180 - threshold}" />
-	<property name="joint_5_limit_soft" value="${M_PI * (167.5 + 167.5) / 180 - threshold}" />
+	<xacro:property name="joint_1_limit" value="${M_PI * (169 + 169) / 180}" />
+	<xacro:property name="joint_2_limit" value="${M_PI * (90 + 65) / 180}" />
+	<xacro:property name="joint_3_limit" value="${M_PI * (146 + 151) / 180}" />
+	<xacro:property name="joint_4_limit" value="${M_PI * (102.5 + 102.5) / 180}" />
+	<xacro:property name="joint_5_limit" value="${M_PI * (167.5 + 167.5) / 180}" />
+        <xacro:property name="joint_1_limit_soft" value="${M_PI * (169 + 169) / 180 - threshold}" />
+	<xacro:property name="joint_2_limit_soft" value="${M_PI * (90 + 65) / 180 - threshold}" />
+	<xacro:property name="joint_3_limit_soft" value="${M_PI * (146 + 151) / 180 - threshold}" />
+	<xacro:property name="joint_4_limit_soft" value="${M_PI * (102.5 + 102.5) / 180 - threshold}" />
+	<xacro:property name="joint_5_limit_soft" value="${M_PI * (167.5 + 167.5) / 180 - threshold}" />
 	<!-- dynamic properties : mass (kg) Alu data sheet -->
-	<property name="link_0_mass" value="0.845" />
-	<property name="link_1_mass" value="2.412" />
-	<property name="link_2_mass" value="1.155" />
-	<property name="link_3_mass" value="0.934" />
-	<property name="link_4_mass" value="0.877" />
-	<property name="link_5_mass" value="0.251" />
-	<!--<property name="link_0_mass" value="0.845" />
-	<property name="link_1_mass" value="0.1" />
-	<property name="link_2_mass" value="0.1" />
-	<property name="link_3_mass" value="0.1" />
-	<property name="link_4_mass" value="0.1" />
-	<property name="link_5_mass" value="0.1" />-->
+	<xacro:property name="link_0_mass" value="0.845" />
+	<xacro:property name="link_1_mass" value="2.412" />
+	<xacro:property name="link_2_mass" value="1.155" />
+	<xacro:property name="link_3_mass" value="0.934" />
+	<xacro:property name="link_4_mass" value="0.877" />
+	<xacro:property name="link_5_mass" value="0.251" />
+	<!--<xacro:property name="link_0_mass" value="0.845" />
+	<xacro:property name="link_1_mass" value="0.1" />
+	<xacro:property name="link_2_mass" value="0.1" />
+	<xacro:property name="link_3_mass" value="0.1" />
+	<xacro:property name="link_4_mass" value="0.1" />
+	<xacro:property name="link_5_mass" value="0.1" />-->
 	<!-- TODO: add inertia tensor-->
 	<xacro:macro name="default_origin">

File: urdf/youbot_base/base.transmission.xacro (robot description, xacro)
@@ -4,92 +4,91 @@
        xmlns:interface="http://playerstage.sourceforge.net/gazebo/xmlschema/#interface"
        xmlns:xacro="http://ros.org/wiki/xacro">
-	<property name="wheel_mechanical_reduction" value="${624/35 * 80/18}" />
-	<property name="caster_mechanical_reduction" value="${624/35 * 80/18}" />
-	<property name="" value="0.360" />
+	<xacro:property name="wheel_mechanical_reduction" value="${624/35 * 80/18}" />
+	<xacro:property name="caster_mechanical_reduction" value="${624/35 * 80/18}" />
 	<xacro:macro name="youbot_base_transmission">
-		<!-- front left wheel -->
+	<!-- front left wheel -->
 		<transmission name="wheel_trans_fl">
-			<type>transmission_interface/SimpleTransmission</type>
+      <type>transmission_interface/SimpleTransmission</type>
 			<actuator name="wheel_motor_fl">
-				<hardwareInterface>VelocityJointInterface</hardwareInterface>
-				<mechanicalReduction>${wheel_mechanical_reduction}</mechanicalReduction>
-			</actuator>
+        <hardwareInterface>VelocityJointInterface</hardwareInterface>
+        <mechanicalReduction>${wheel_mechanical_reduction}</mechanicalReduction>
+      </actuator>
 			<joint name="wheel_joint_fl">
-				<hardwareInterface>VelocityJointInterface</hardwareInterface>
-			</joint>
+        <hardwareInterface>VelocityJointInterface</hardwareInterface>
+      </joint>
 		</transmission>
 		<transmission name="caster_trans_fl">
-			<type>transmission_interface/SimpleTransmission</type>
-			<actuator name="caster_motor_fl">
-				<hardwareInterface>VelocityJointInterface</hardwareInterface>
-				<mechanicalReduction>${caster_mechanical_reduction}</mechanicalReduction>
-			</actuator>
-			<joint name="caster_joint_fl">
-				<hardwareInterface>VelocityJointInterface</hardwareInterface>
-			</joint>
-		</transmission>
-		<!-- front right wheel -->
-		<transmission name="wheel_trans_fr">
-			<type>transmission_interface/SimpleTransmission</type>
-			<actuator name="wheel_motor_fr">
-				<hardwareInterface>VelocityJointInterface</hardwareInterface>
-				<mechanicalReduction>${wheel_mechanical_reduction}</mechanicalReduction>
-			</actuator>
-			<joint name="wheel_joint_fr">
-				<hardwareInterface>VelocityJointInterface</hardwareInterface>
-			</joint>
-		</transmission>
-		<transmission name="caster_trans_fr">
-			<type>transmission_interface/SimpleTransmission</type>
-			<actuator name="caster_motor_fr" >
-				<hardwareInterface>VelocityJointInterface</hardwareInterface>
-				<mechanicalReduction>${caster_mechanical_reduction}</mechanicalReduction>
-			</actuator>
-			<joint name="caster_joint_fr">
-				<hardwareInterface>VelocityJointInterface</hardwareInterface>
-			</joint>
-		</transmission>
-		<!-- back left wheel -->
-		<transmission name="wheel_trans_bl">
-			<type>transmission_interface/SimpleTransmission</type>
-			<actuator name="wheel_motor_bl" >
-				<hardwareInterface>VelocityJointInterface</hardwareInterface>
-				<mechanicalReduction>${wheel_mechanical_reduction}</mechanicalReduction>
-			</actuator>
-			<joint name="wheel_joint_bl">
-				<hardwareInterface>VelocityJointInterface</hardwareInterface>
-			</joint>
-		</transmission>
-		<transmission name="caster_trans_bl">
-			<type>transmission_interface/SimpleTransmission</type>
-			<actuator name="caster_motor_bl" >
-				<hardwareInterface>VelocityJointInterface</hardwareInterface>
-				<mechanicalReduction>${caster_mechanical_reduction}</mechanicalReduction>
-			</actuator>
-			<joint name="caster_joint_bl">
-				<hardwareInterface>VelocityJointInterface</hardwareInterface>
-			</joint>
-		</transmission>
-		<!-- back right wheel -->
-		<transmission name="wheel_trans_br">
-			<type>transmission_interface/SimpleTransmission</type>
-			<actuator name="wheel_motor_br" >
-				<hardwareInterface>VelocityJointInterface</hardwareInterface>
-				<mechanicalReduction>${wheel_mechanical_reduction}</mechanicalReduction>
-			</actuator>
-			<joint name="wheel_joint_br">
-				<hardwareInterface>VelocityJointInterface</hardwareInterface>
-			</joint>
-		</transmission>
-		<transmission name="caster_trans_br">
-			<type>transmission_interface/SimpleTransmission</type>
-			<actuator name="caster_motor_br" >
-				<hardwareInterface>VelocityJointInterface</hardwareInterface>
-				<mechanicalReduction>${caster_mechanical_reduction}</mechanicalReduction>
-			</actuator>
-			<joint name="caster_joint_br">
-				<hardwareInterface>VelocityJointInterface</hardwareInterface>
-			</joint>
-		</transmission>
-	</xacro:macro>
+      <type>transmission_interface/SimpleTransmission</type>
+   	  <actuator name="caster_motor_fl">
+        <hardwareInterface>VelocityJointInterface</hardwareInterface>
+        <mechanicalReduction>${caster_mechanical_reduction}</mechanicalReduction>
+      </actuator>
+      <joint name="caster_joint_fl">
+        <hardwareInterface>VelocityJointInterface</hardwareInterface>
+      </joint>
+    </transmission>
+	  <!-- front right wheel -->
+	  <transmission name="wheel_trans_fr">
+      <type>transmission_interface/SimpleTransmission</type>
+		  <actuator name="wheel_motor_fr">
+        <hardwareInterface>VelocityJointInterface</hardwareInterface>
+        <mechanicalReduction>${wheel_mechanical_reduction}</mechanicalReduction>
+      </actuator>
+		  <joint name="wheel_joint_fr">
+        <hardwareInterface>VelocityJointInterface</hardwareInterface>
+      </joint>
+	  </transmission>
+	  <transmission name="caster_trans_fr">
+      <type>transmission_interface/SimpleTransmission</type>
+      <actuator name="caster_motor_fr" >
+        <hardwareInterface>VelocityJointInterface</hardwareInterface>
+        <mechanicalReduction>${caster_mechanical_reduction}</mechanicalReduction>
+      </actuator>
+      <joint name="caster_joint_fr">
+        <hardwareInterface>VelocityJointInterface</hardwareInterface>
+      </joint>
+    </transmission>
+	  <!-- back left wheel -->
+	  <transmission name="wheel_trans_bl">
+      <type>transmission_interface/SimpleTransmission</type>
+	    <actuator name="wheel_motor_bl" >
+        <hardwareInterface>VelocityJointInterface</hardwareInterface>
+        <mechanicalReduction>${wheel_mechanical_reduction}</mechanicalReduction>
+      </actuator>
+	    <joint name="wheel_joint_bl">
+        <hardwareInterface>VelocityJointInterface</hardwareInterface>
+      </joint>
+	  </transmission>
+	  <transmission name="caster_trans_bl">
+      <type>transmission_interface/SimpleTransmission</type>
+      <actuator name="caster_motor_bl" >
+        <hardwareInterface>VelocityJointInterface</hardwareInterface>
+        <mechanicalReduction>${caster_mechanical_reduction}</mechanicalReduction>
+      </actuator>
+      <joint name="caster_joint_bl">
+        <hardwareInterface>VelocityJointInterface</hardwareInterface>
+      </joint>
+    </transmission>
+	  <!-- back right wheel -->
+	  <transmission name="wheel_trans_br">
+      <type>transmission_interface/SimpleTransmission</type>
+	    <actuator name="wheel_motor_br" >
+        <hardwareInterface>VelocityJointInterface</hardwareInterface>
+        <mechanicalReduction>${wheel_mechanical_reduction}</mechanicalReduction>
+      </actuator>
+		  <joint name="wheel_joint_br">
+        <hardwareInterface>VelocityJointInterface</hardwareInterface>
+      </joint>
+	  </transmission>
+	  <transmission name="caster_trans_br">
+      <type>transmission_interface/SimpleTransmission</type>
+      <actuator name="caster_motor_br" >
+        <hardwareInterface>VelocityJointInterface</hardwareInterface>
+        <mechanicalReduction>${caster_mechanical_reduction}</mechanicalReduction>
+      </actuator>
+      <joint name="caster_joint_br">
+        <hardwareInterface>VelocityJointInterface</hardwareInterface>
+      </joint>
+    </transmission>
+  </xacro:macro>
 </robot>

File: urdf/youbot_base/base.urdf.xacro (robot description, xacro)
@@ -8,28 +8,28 @@
   <xacro:include filename="$(find youbot_description)/urdf/youbot_base/base.transmission.xacro"/>
   <!-- simplified box collision geometry for base -->
-  <property name="base_size_x" value="0.570"/>
-  <property name="base_size_y" value="0.360"/>
-  <property name="base_size_z" value="0.100"/>
-  <property name="base_mass" value="22.0"/>
-  <property name="caster_offset_x" value="0.228"/>
-  <property name="caster_offset_y" value="0.158"/>
-  <property name="caster_offset_z" value="-0.034"/>
-  <property name="caster_mass" value="0.1"/>
-  <property name="wheel_offset_x" value="0.0"/>
-  <property name="wheel_offset_y" value="0.0"/>
-  <property name="wheel_offset_z" value="0.0"/>
-  <property name="wheel_mass" value="0.4"/>
-  <property name="wheel_radius" value="0.05"/>
-  <property name="wheel_length" value="0.005"/>
-  <property name="caster_joint_damping" value="1.0"/>
-  <property name="caster_joint_friction" value="1.0"/>
-  <property name="caster_joint_effort" value="30"/>
-  <property name="caster_joint_velocity" value="10"/>
-  <property name="caster_joint_safety_k_velocity" value="10.0"/>
-  <property name="wheel_joint_damping" value="1.0"/>
-  <property name="wheel_joint_friction" value="1.0"/>
-  <property name="wheel_joint_effort" value="30"/>
-  <property name="wheel_joint_velocity" value="10"/>
-  <property name="wheel_joint_safety_k_velocity" value="10.0"/>
+  <xacro:property name="base_size_x" value="0.570"/>
+  <xacro:property name="base_size_y" value="0.360"/>
+  <xacro:property name="base_size_z" value="0.100"/>
+  <xacro:property name="base_mass" value="22.0"/>
+  <xacro:property name="caster_offset_x" value="0.228"/>
+  <xacro:property name="caster_offset_y" value="0.158"/>
+  <xacro:property name="caster_offset_z" value="-0.034"/>
+  <xacro:property name="caster_mass" value="0.1"/>
+  <xacro:property name="wheel_offset_x" value="0.0"/>
+  <xacro:property name="wheel_offset_y" value="0.0"/>
+  <xacro:property name="wheel_offset_z" value="0.0"/>
+  <xacro:property name="wheel_mass" value="0.4"/>
+  <xacro:property name="wheel_radius" value="0.05"/>
+  <xacro:property name="wheel_length" value="0.005"/>
+  <xacro:property name="caster_joint_damping" value="1.0"/>
+  <xacro:property name="caster_joint_friction" value="1.0"/>
+  <xacro:property name="caster_joint_effort" value="30"/>
+  <xacro:property name="caster_joint_velocity" value="10"/>
+  <xacro:property name="caster_joint_safety_k_velocity" value="10.0"/>
+  <xacro:property name="wheel_joint_damping" value="1.0"/>
+  <xacro:property name="wheel_joint_friction" value="1.0"/>
+  <xacro:property name="wheel_joint_effort" value="30"/>
+  <xacro:property name="wheel_joint_velocity" value="10"/>
+  <xacro:property name="wheel_joint_safety_k_velocity" value="10.0"/>
   <xacro:macro name="youbot_base" params="name">
     <link name="${name}_footprint">
