Commit message: added hokuyo scanner

File: urdf/youbot_gripper/gripper.transmission.xacro (robot description, xacro)
@@ -6,22 +6,22 @@
 	<xacro:macro name="youbot_gripper_transmission" params="name">
 		<transmission name="${name}_finger_l_trans">
-			<type>transmission_interface/SimpleTransmission</type>
+      <type>transmission_interface/SimpleTransmission</type>
 			<actuator name="${name}_finger_l_motor">
-				<hardwareInterface>EffortJointInterface</hardwareInterface>
-				<mechanicalReduction>1</mechanicalReduction>
-			</actuator>
+        <hardwareInterface>EffortJointInterface</hardwareInterface>
+        <mechanicalReduction>1</mechanicalReduction>
+      </actuator>
 			<joint name="${name}_finger_joint_l">
-				<hardwareInterface>EffortJointInterface</hardwareInterface>
-			</joint>
+        <hardwareInterface>EffortJointInterface</hardwareInterface>
+      </joint>
 		</transmission>
 		<transmission name="${name}_finger_r_trans">
-			<type>transmission_interface/SimpleTransmission</type>
+      <type>transmission_interface/SimpleTransmission</type>
 			<actuator name="${name}_finger_r_motor">
-				<hardwareInterface>EffortJointInterface</hardwareInterface>
-				<mechanicalReduction>1</mechanicalReduction>
-			</actuator>
+        <hardwareInterface>EffortJointInterface</hardwareInterface>
+        <mechanicalReduction>1</mechanicalReduction>
+      </actuator>
 			<joint name="${name}_finger_joint_r">
-				<hardwareInterface>EffortJointInterface</hardwareInterface>
-			</joint>
+        <hardwareInterface>EffortJointInterface</hardwareInterface>
+      </joint>
 		</transmission>
 	</xacro:macro>

File: urdf/youbot_gripper/gripper.urdf.xacro (robot description, xacro)
@@ -10,5 +10,5 @@
 		<!-- joint between arm_7_link and sdh_palm_link -->
 		<joint name="${name}_palm_joint" type="fixed" >
-			<insert_block name="origin" />
+			<xacro:insert_block name="origin" />
 			<parent link="${parent}" />
 			<child link="${name}_palm_link" />

File: urdf/youbot_gripper/limits.urdf.xacro (robot description, xacro)
@@ -1,9 +1,9 @@
 <?xml version="1.0"?>
-<robot>
+<robot xmlns:xacro="http://ros.org/wiki/xacro">
 	<!-- common properties -->
-	<property name="M_PI" value="3.1415926535897931" />
-        <property name="threshold" value="0.001" />
+	<xacro:property name="M_PI" value="3.1415926535897931" />
+        <xacro:property name="threshold" value="0.001" />
 	<!-- fingers limits, values are in meters -->
-	<property name="finger_joint" value="${0.023 / 2.0}" />
-	<property name="finger_joint_soft" value="${(0.023 - threshold) / 2.0}" />
+	<xacro:property name="finger_joint" value="${0.023 / 2.0}" />
+	<xacro:property name="finger_joint_soft" value="${(0.023 - threshold) / 2.0}" />
 </robot>

File: urdf/youbot_plate/plate.urdf.xacro (robot description, xacro)
@@ -7,5 +7,5 @@
 		<!-- joint between arm_7_link and sdh_palm_link -->
 		<joint name="${name}_joint" type="fixed" >
-			<insert_block name="origin" />
+			<xacro:insert_block name="origin" />
 			<parent link="${parent}" />
 			<child link="${name}_link" />
